File: hardware/kicad/bwlr1c.kicad_sch (KiCad schematic)
At the start: 35 parts, among them J1 Program, J2 Debug, Q1 AO3407, SW3 RESET, SW4 BOOT, U1 BME680, U2 RAK3172

Commit message: upload resources
Other:
- company: (none) -> Teapot Laboratories
- title: (none) -> Teapot BWLR1C
Changed lines of the file:
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@@
 (kicad_sch (version 20211123) (generator eeschema)
   (paper "A4")
+  (title_block
+    (title "Teapot BWLR1C")
+    (date "2022-08-24")
+    (rev "1")
+    (company "Teapot Laboratories")
+  )
   (junction (at 80.01 64.77) (diameter 0) (color 0 0 0 0)
   )
